File: pcb/DivaConIO/DivaConIO.kicad_pcb (KiCad board)
At the start: 2 copper layers, 55.9 x 70.5 mm, 34 parts, among them J1 DPad Buttons, J10 SWD, J2 Slider i2c, J3 Display i2c, J4 Face Buttons, J5 Button LEDs, J6 L Buttons, J7 Fn Buttons, J8 R Buttons, J9 Slider LEDs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

Commit message: DivaConIO revision 2
- Changed JP1 to allow external power supply
- Added +5V to empty pin on SWD connector
Parts:
- added JP2: Bridge LED Data, Jumper:SolderJumper-2_P1.3mm_Open_RoundedPad1.0x1.5mm, F.Cu at (160.0, 72.0)
- moved JP1 2.54 mm to (158.2, 50.8), turned to 180 degrees
Connections:
- J10 pad 2: unconnected-(J10-Pin_2-Pad2) -> +5V
- JP1 pad 1: Net-(JP1-A) -> +5V
- JP1 pad 2: +5V -> Net-(JP1-B)
- U1 pad 39: Net-(JP1-A) -> +5V
- U1 pad 40: +5V -> Net-(JP1-B)
Routing:
- net +5V: track 119.8 -> 129.3 mm, vias 0 -> 1
- net Net-(JP1-B): track 0.00 -> 6.46 mm
- net Net-(JP1-A): track 6.32 -> 0.00 mm
- net Net-(J9-Pin_4): track 15.7 -> 18.1 mm
- net Slider LED Data: track 9.14 -> 11.6 mm
