File: pcb/DivaConSliderCap/DivaConSlider.kicad_pcb (KiCad board)
At the start: 2 copper layers, 548 x 93 mm, 191 parts, among them J1 Slider I2C, J2 Slider LED, J3 Display I2C, J4 Display, U1 CAP1188, U2 CAP1188, U3 CAP1188, U4 CAP1188

Commit message: Move Cap1188 based slider to correctly named subdir
Other:
- board text added: "0x29"
- board text added: "0x2A"
- board text added: "0x2B"
- board text added: "0x2C"
Changed lines of the file:
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@@
+		)
+	)
+	(gr_text "0x2A"
+		(at 359 154 0)
+		(layer "F.SilkS")
+		(effects
+			(font
+				(size 1.5 1.5)
+				(thickness 0.3)
+				(bold yes)
+			)
+			(justify left bottom)
+		)
+	)
+	(gr_text "0x2C"
+		(at 87 154 0)
+		(layer "F.SilkS")
+		(effects
+			(font
+				(size 1.5 1.5)
+				(thickness 0.3)
+				(bold yes)
+			)
+			(justify left bottom)
+		)
+	)
+	(gr_text "0x29"
+		(at 495 154 0)
+		(layer "F.SilkS")
+		(effects
+			(font
+				(size 1.5 1.5)
+				(thickness 0.3)
+				(bold yes)
+			)
+			(justify left bottom)
 		)
 	)
@@
 		)
 	)
-	(gr_text "${TITLE} Rev. ${REVISION}"
-		(at 339.5 141.75 0)
+	(gr_text "0x2B"
+		(at 223 154 0)
 		(layer "F.SilkS")
 		(effects
@@
 		)
 	)
+	(gr_text "${TITLE} Rev. ${REVISION}"
+		(at 339.5 141.75 0)
+		(layer "F.SilkS" knockout)
+		(effects
+			(font
+				(size 1.5 1.5)
+				(thickness 0.3)
+				(bold yes)
+			)
+			(justify left bottom)
+		)
+	)
 	(gr_text "JLCJLCJLCJLC"
-		(at 146.75 162.5 90)
+		(at 66 141 0)
 		(layer "F.SilkS")
 		(effects
